File: BeagleBone_Black_Wireless.sch (EAGLE design)
At the start: 275 parts, among them IC1 OSD3358, IC10 TXS0108ERGYR, IC11 TXS0108ERGYR, IC12 TPS2051BDGN, IC13 SN74AUC1G74, IC14 TPD4S012DRY, IC15 TPD4S012DRY, IC17 SN74LVC2G241DCUR, IC18 TL1963ADCQR, IC19 AP2112K-1.8TRG1 3.3V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

Commit message: Add rev A5 source files
Parts:
- C2: value .1uF,6.3V -> .1uF, 6.3V
- FB2: value 150 Ohm 800mA -> 2.5k Ohm (BLM18BD252SN1D)
- FB5, FB6: value 33 -> 1k BLM15AG102SN1D
- FB7: value 0, 1% -> 1k BLM15AG102SN1D
- renumbered JTAG1 to P2, R113 to FB6, R15 to FB7, R9 to FB5, X8 to P8, X9 to P9
Connections:
- net MCC1_CLK renamed MMC1_CLK
- net MCC1_CMD renamed MMC1_CMD
- net MCC1_DAT0 renamed MMC1_DAT0
- net MCC1_DAT1 renamed MMC1_DAT1
- net MCC1_DAT2 renamed MMC1_DAT2
- net MCC1_DAT3 renamed MMC1_DAT3
- net MCC1_DAT4 renamed MMC1_DAT4
- net MCC1_DAT5 renamed MMC1_DAT5
- net MCC1_DAT6 renamed MMC1_DAT6
- net MCC1_DAT7 renamed MMC1_DAT7
Other:
- note added: "A5"
- note added: "GHI-PROTO-BBBW-REV-A5"
- note removed: "A3"
- note removed: "GHI-PROTO-BBBW-REV-A3"
