File: EAGLE/BeagleBone_Black_Wireless.sch (EAGLE design)
At the start: 275 parts, among them IC1 OSD3358, IC10 TXS0108ERGYR, IC11 TXS0108ERGYR, IC12 TPS2051BDGN, IC13 SN74AUC1G74, IC14 TPD4S012DRY, IC15 TPD4S012DRY, IC17 SN74LVC2G241DCUR, IC18 TL1963ADCQR, IC19 AP2112K-1.8TRG1 3.3V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

Commit message: PCB rev A5b: Added vias to pads
This is meant to assist in avoiding pads coming off with excess pressure.
Parts:
- IC6: value TLVH431 (SOT-23-3) -> DNP TLVH431 (SOT-23-3)
- R48: value 499 -> DNP 499
- R50: value 10k 1% -> DNP 10k 1%
- R51: value 40.2k 1% -> DNP 40.2k 1%
- R56: value 1M, 1% -> DNP 1M, 1%
- T2: value MMBT2907 -> DNP MMBT2907
- X12: value PJ-102B_POWER_CON -> (none); device GHI:PJ-102B_POWER_CON -> GHI-Connectors:PJ-102B_POWER_CON
Changed lines of the file:
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@@
 <part name="GND6" library="supply1" deviceset="GND" device=""/>
 <part name="IC5" library="texas" deviceset="LM4041*I" device="DBZ" technology="D" value="TLVH431 (SOT-23-3)"/>
-<part name="IC6" library="texas" deviceset="LM4041*I" device="DBZ" technology="D" value="TLVH431 (SOT-23-3)"/>
+<part name="IC6" library="texas" deviceset="LM4041*I" device="DBZ" technology="D" value="DNP TLVH431 (SOT-23-3)"/>
 <part name="SUPPLY33" library="GHI-PowerGoundSupply" deviceset="VDD_3V3A" device=""/>
 <part name="SUPPLY34" library="GHI-PowerGoundSupply" deviceset="VDD_1V8" device=""/>
 <part name="SUPPLY38" library="GHI-PowerGoundSupply" deviceset="VDD_3V3B" device=""/>
 <part name="R44" library="rcl" deviceset="R-US_" device="R0402" value="499"/>
-<part name="R48" library="rcl" deviceset="R-US_" device="R0402" value="499"/>
+<part name="R48" library="rcl" deviceset="R-US_" device="R0402" value="DNP 499"/>
 <part name="R46" library="rcl" deviceset="R-US_" device="R0402" value="10k 1%"/>
-<part name="R50" library="rcl" deviceset="R-US_" device="R0402" value="10k 1%"/>
-<part name="R51" library="rcl" deviceset="R-US_" device="R0402" value="40.2k 1%"/>
+<part name="R50" library="rcl" deviceset="R-US_" device="R0402" value="DNP 10k 1%"/>
+<part name="R51" library="rcl" deviceset="R-US_" device="R0402" value="DNP 40.2k 1%"/>
 <part name="R47" library="rcl" deviceset="R-US_" device="R0402" value="40.2k 1%"/>
 <part name="R45" library="rcl" deviceset="R-US_" device="R0402" value="DNP"/>
@@
 <part name="SUPPLY2" library="GHI-PowerGoundSupply" deviceset="VDD_3V3B" device=""/>
 <part name="T1" library="transistor-pnp" deviceset="MMBT2907*" device="SMD" technology="ALT1" value="MMBT2907"/>
-<part name="T2" library="transistor-pnp" deviceset="MMBT2907*" device="SMD" technology="ALT1" value="MMBT2907"/>
+<part name="T2" library="transistor-pnp" deviceset="MMBT2907*" device="SMD" technology="ALT1" value="DNP MMBT2907"/>
 <part name="GND68" library="supply1" deviceset="GND" device=""/>
-<part name="X12" library="GHI" deviceset="PJ-102B_POWER_CON" device=""/>
 <part name="GND33" library="supply1" deviceset="GND" device=""/>
 <part name="FUD4" library="GHI" deviceset="FIDUCIAL" device=""/>
@@
 <part name="GND5" library="supply1" deviceset="GND" device=""/>
 <part name="C23" library="rcl" deviceset="CPOL-US" device="CT3528" value="47uF DNP"/>
-<part name="R56" library="rcl" deviceset="R-US_" device="R0402" value="1M, 1%"/>
+<part name="R56" library="rcl" deviceset="R-US_" device="R0402" value="DNP 1M, 1%"/>
+<part name="X12" library="GHI-Connectors" deviceset="PJ-102B_POWER_CON" device=""/>
 </parts>
 <sheets>
@@
 </instance>
 <instance part="GND68" gate="1" x="604.52" y="548.64"/>
-<instance part="X12" gate="G$1" x="596.9" y="558.8"/>
 <instance part="GND33" gate="1" x="807.72" y="83.82"/>
 <instance part="FUD4" gate="G$1" x="787.4" y="48.26"/>
@@
 </instance>
 <instance part="R56" gate="G$1" x="43.18" y="518.16" rot="R90"/>
+<instance part="X12" gate="G$1" x="596.9" y="558.8"/>
 </instances>
 <busses>
@@
 <pinref part="GND68" gate="1" pin="GND"/>
 <wire x1="604.52" y1="551.18" x2="604.52" y2="553.72" width="0.1524" layer="91"/>
-<pinref part="X12" gate="G$1" pin="OUT"/>
-<wire x1="604.52" y1="553.72" x2="601.98" y2="553.72" width="0.1524" layer="91"/>
 <pinref part="R17" gate="G$1" pin="1"/>
 <wire x1="607.06" y1="553.72" x2="604.52" y2="553.72" width="0.1524" layer="91"/>
 <junction x="604.52" y="553.72"/>
+<pinref part="X12" gate="G$1" pin="OUT"/>
+<wire x1="604.52" y1="553.72" x2="601.98" y2="553.72" width="0.1524" layer="91"/>
 </segment>
 <segment>
@@
 <wire x1="637.54" y1="558.8" x2="640.08" y2="558.8" width="0.1524" layer="91"/>
 <junction x="637.54" y="558.8"/>
-<pinref part="X12" gate="G$1" pin="IN"/>
 <wire x1="601.98" y1="558.8" x2="637.54" y2="558.8" width="0.1524" layer="91"/>
+<pinref part="X12" gate="G$1" pin="IN"/>
 </segment>
 <segment>
